File: untitled.kicad_sch (KiCad schematic)
At the start: 4 parts, among them J1 I2C, J2 ICSP, J3 Serial UART, J4 GPIO

Commit message: fixed SCL and SCK
Connections:
- net SCL: no longer J2.3 (Pin_3)
- new net SCK: J2.3 (Pin_3)
Changed lines of the file:
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@@
 		)
 	)
-	(hierarchical_label "SCL"
+	(hierarchical_label "SCK"
 		(shape passive)
 		(at 119.38 107.95 180)
